File: hardware/schematics/top_level.kicad_sch (KiCad schematic)
At the start: 3 parts

Commit message: fix(hardware): fully migrate schematics to native KiCad 10 syntax and pass ERC
Parts:
- removed ?: (no value), symbol custom_power:VDD
- removed ?: (no value), symbol custom_power:VSS
- removed ?: (no value), symbol custom_power:GND
