File: hardware/schematics/adex_neuron_cell.kicad_sch (KiCad schematic)
At the start: 13 parts

Commit message: fix(hardware): fully migrate schematics to native KiCad 10 syntax and pass ERC
Parts:
- removed ?: (no value), symbol custom_power:VDD
- removed ?: (no value), symbol custom_power:VSS
- removed ?: (no value), symbol custom_power:GND
- C1: renamed from ?; value (none) -> 10nF; footprint (none) -> Capacitor_SMD:C_0805_2012Metric; ['name', 'Datasheet'] ['value', ''] -> (none); ['name', 'Footprint'] ['value', 'Capacitor_SMD:C_0805_2012Metric'] -> (none); ['name', 'Reference'] ['value', 'C1'] -> (none); ['name', 'Value'] ['value', '10nF'] -> (none); ['name', 'ki_description'] ['value', 'Membrane capacitor, C0G/NP0, 0805'] -> (none)
- Q1: renamed from ?; value (none) -> 2N3904; footprint (none) -> Package_TO_SOT_SMD:SOT-23; ['name', 'Datasheet'] ['value', 'https://www.onsemi.com/pdf/datasheet/2n3903-d.pd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 -> (none); ['name', 'Footprint'] ['value', 'Package_TO_SOT_SMD:SOT-23'] -> (none); ['name', 'Reference'] ['value', 'Q1'] -> (none); ['name', 'Value'] ['value', '2N3904'] -> (none); ['name', 'ki_description'] ['value', 'NPN BJT SOT-23 exponential current source'] -> (none)
- Q2: renamed from ?; value (none) -> BSS138; footprint (none) -> Package_TO_SOT_SMD:SOT-23; ['name', 'Datasheet'] ['value', 'https://www.onsemi.com/pdf/datasheet/bss138-d.pd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 -> (none); ['name', 'Footprint'] ['value', 'Package_TO_SOT_SMD:SOT-23'] -> (none); ['name', 'Reference'] ['value', 'Q2'] -> (none); ['name', 'Value'] ['value', 'BSS138'] -> (none); ['name', 'ki_description'] ['value', 'N-Ch MOSFET SOT-23 membrane reset switch'] -> (none)
- R1: renamed from ?; value (none) -> 10M; footprint (none) -> Resistor_SMD:R_0805_2012Metric; ['name', 'Datasheet'] ['value', ''] -> (none); ['name', 'Footprint'] ['value', 'Resistor_SMD:R_0805_2012Metric'] -> (none); ['name', 'Reference'] ['value', 'R1'] -> (none); ['name', 'Value'] ['value', '10M'] -> (none); ['name', 'ki_description'] ['value', 'Leak resistance, 10 MOhm, 0805'] -> (none)
- R2: renamed from ?; value (none) -> 1k; footprint (none) -> Resistor_SMD:R_0805_2012Metric; ['name', 'Datasheet'] ['value', ''] -> (none); ['name', 'Footprint'] ['value', 'Resistor_SMD:R_0805_2012Metric'] -> (none); ['name', 'Reference'] ['value', 'R2'] -> (none); ['name', 'Value'] ['value', '1k'] -> (none)
- R3: renamed from ?; value (none) -> 100; footprint (none) -> Resistor_SMD:R_0805_2012Metric; ['name', 'Datasheet'] ['value', ''] -> (none); ['name', 'Footprint'] ['value', 'Resistor_SMD:R_0805_2012Metric'] -> (none); ['name', 'Reference'] ['value', 'R3'] -> (none); ['name', 'Value'] ['value', '100'] -> (none)
- R4: renamed from ?; value (none) -> 100k; footprint (none) -> Resistor_SMD:R_0805_2012Metric; ['name', 'Datasheet'] ['value', ''] -> (none); ['name', 'Footprint'] ['value', 'Resistor_SMD:R_0805_2012Metric'] -> (none); ['name', 'Reference'] ['value', 'R4'] -> (none); ['name', 'Value'] ['value', '100k'] -> (none)
- R5: renamed from ?; value (none) -> 100k; footprint (none) -> Resistor_SMD:R_0805_2012Metric; ['name', 'Datasheet'] ['value', ''] -> (none); ['name', 'Footprint'] ['value', 'Resistor_SMD:R_0805_2012Metric'] -> (none); ['name', 'Reference'] ['value', 'R5'] -> (none); ['name', 'Value'] ['value', '100k'] -> (none)
- R6: renamed from ?; value (none) -> 10k; footprint (none) -> Resistor_SMD:R_0805_2012Metric; ['name', 'Datasheet'] ['value', ''] -> (none); ['name', 'Footprint'] ['value', 'Resistor_SMD:R_0805_2012Metric'] -> (none); ['name', 'Reference'] ['value', 'R6'] -> (none); ['name', 'Value'] ['value', '10k'] -> (none)
- U1: renamed from ?; value (none) -> LM393; footprint (none) -> Package_SO:SOIC-8_3.9x4.9mm_P1.27mm; ['name', 'Datasheet'] ['value', 'https://www.ti.com/lit/ds/symlink/lm393.pdf'] -> (none); ['name', 'Footprint'] ['value', 'Package_SO:SOIC-8_3.9x4.9mm_P1.27mm'] -> (none); ['name', 'Reference'] ['value', 'U1'] -> (none); ['name', 'Value'] ['value', 'LM393'] -> (none); ['name', 'ki_description'] ['value', 'Low-power open-collector comparator SOIC-8'] -> (none)

Commit message: fix(hardware): unify KiCad project hierarchy and link schematic netlist to PCB layout
Parts:
- Q1: symbol Device:Q_NPN_BCE -> Transistor_BJT:Q_NPN_BCE
Changed lines of the file:
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@@
   ;; ──────────────────────────────────────────────
   (symbol
-    (lib_id "Device:Q_NPN_BCE")
+    (lib_id "Transistor_BJT:Q_NPN_BCE")
     (at 150 400 0)
     (unit 1)

Commit message: refactor(hardware): shrink footprints to 0402/TSSOP-8 and expand routing corridors across 70x70mm PCB
Parts:
- C1: footprint Capacitor_SMD:C_0805_2012Metric -> Capacitor_SMD:C_0402_1005Metric
- R1, R2, R3, R4, R5, R6: footprint Resistor_SMD:R_0805_2012Metric -> Resistor_SMD:R_0402_1005Metric
- U1: footprint Package_SO:SOIC-8_3.9x4.9mm_P1.27mm -> Package_SO:TSSOP-8_4.4x3mm_P0.65mm
Changed lines of the file:
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@@
   )
   ;; ──────────────────────────────────────────────
-  ;;  COMPONENT: INTEGRATOR — C_m  (10 nF, 0805, C0G/NP0)
+  ;;  COMPONENT: INTEGRATOR — C_m  (10 nF, 0603, C0G/NP0)
   ;; ──────────────────────────────────────────────
   (symbol
@@
       (effects (font (size 1.27 1.27)))
     )
-    (property "Footprint" "Capacitor_SMD:C_0805_2012Metric"
-      (at 180 250 0)
-      (effects (font (size 1.27 1.27)) (hide yes))
-    )
-    (property "Datasheet" ""
-      (at 180 250 0)
-      (effects (font (size 1.27 1.27)) (hide yes))
-    )
-    (property "ki_description" "Membrane capacitor, C0G/NP0, 0805"
-      (at 180 250 0)
-      (effects (font (size 1.27 1.27)))
-    )
-  )
-  ;; ──────────────────────────────────────────────
-  ;;  COMPONENT: INTEGRATOR — R_L  (10 MΩ, 0805)
+    (property "Footprint" "Capacitor_SMD:C_0402_1005Metric"
+      (at 180 250 0)
+      (effects (font (size 1.27 1.27)) (hide yes))
+    )
+    (property "Datasheet" ""
+      (at 180 250 0)
+      (effects (font (size 1.27 1.27)) (hide yes))
+    )
+    (property "ki_description" "Membrane capacitor, C0G/NP0, 0402"
+      (at 180 250 0)
+      (effects (font (size 1.27 1.27)))
+    )
+  )
+  ;; ──────────────────────────────────────────────
+  ;;  COMPONENT: INTEGRATOR — R_L  (10 MΩ, 0603)
   ;; ──────────────────────────────────────────────
   (symbol
@@
       (effects (font (size 1.27 1.27)))
     )
-    (property "Footprint" "Resistor_SMD:R_0805_2012Metric"
-      (at 280 250 0)
-      (effects (font (size 1.27 1.27)) (hide yes))
-    )
-    (property "Datasheet" ""
-      (at 280 250 0)
-      (effects (font (size 1.27 1.27)) (hide yes))
-    )
-    (property "ki_description" "Leak resistance, 10 MOhm, 0805"
+    (property "Footprint" "Resistor_SMD:R_0402_1005Metric"
+      (at 280 250 0)
+      (effects (font (size 1.27 1.27)) (hide yes))
+    )
+    (property "Datasheet" ""
+      (at 280 250 0)
+      (effects (font (size 1.27 1.27)) (hide yes))
+    )
+    (property "ki_description" "Leak resistance, 10 MOhm, 0402"
       (at 280 250 0)
       (effects (font (size 1.27 1.27)))
@@
       (effects (font (size 1.27 1.27)))
     )
-    (property "Footprint" "Package_SO:SOIC-8_3.9x4.9mm_P1.27mm"
+    (property "Footprint" "Package_SO:TSSOP-8_4.4x3mm_P0.65mm"
       (at 350 400 0)
       (effects (font (size 1.27 1.27)) (hide yes))
@@
       (effects (font (size 1.27 1.27)) (hide yes))
     )
-    (property "ki_description" "Low-power open-collector comparator SOIC-8"
+    (property "ki_description" "Low-power open-collector comparator TSSOP-8"
       (at 350 400 0)
       (effects (font (size 1.27 1.27)))
@@
       (effects (font (size 1.27 1.27)))
     )
-    (property "Footprint" "Resistor_SMD:R_0805_2012Metric"
+    (property "Footprint" "Resistor_SMD:R_0402_1005Metric"
       (at 150 480 0)
       (effects (font (size 1.27 1.27)) (hide yes))
@@
       (effects (font (size 1.27 1.27)))
     )
-    (property "Footprint" "Resistor_SMD:R_0805_2012Metric"
+    (property "Footprint" "Resistor_SMD:R_0402_1005Metric"
       (at 100 540 0)
       (effects (font (size 1.27 1.27)) (hide yes))
@@
       (effects (font (size 1.27 1.27)))
     )
-    (property "Footprint" "Resistor_SMD:R_0805_2012Metric"
+    (property "Footprint" "Resistor_SMD:R_0402_1005Metric"
       (at 300 550 0)
       (effects (font (size 1.27 1.27)) (hide yes))
@@
       (effects (font (size 1.27 1.27)))
     )
-    (property "Footprint" "Resistor_SMD:R_0805_2012Metric"
+    (property "Footprint" "Resistor_SMD:R_0402_1005Metric"
       (at 350 550 0)
       (effects (font (size 1.27 1.27)) (hide yes))
@@
       (effects (font (size 1.27 1.27)))
     )
-    (property "Footprint" "Resistor_SMD:R_0805_2012Metric"
+    (property "Footprint" "Resistor_SMD:R_0402_1005Metric"
       (at 400 620 0)
       (effects (font (size 1.27 1.27)) (hide yes))
