File: hardware/schematics/lc_bridge_cell.kicad_sch (KiCad schematic)
At the start: 0 parts

Commit message: feat(hardware): define schematic components and complete hierarchical netlist wiring
Parts:
- added ?: (no value)
Changed lines of the file:
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@@
   ;;  Hierarchical Labels — INPUT
   ;; ──────────────────────────────────────────────
-  (hierarchical_label "LC_IN" (shape input) (at 0 50 0)
+  (hierarchical_label "NODE_A" (shape input) (at 50 200 0)
     (fields_autoplaced)
     (font (size 1.27 1.27) (thickness 0.254))
   )
-  (hierarchical_label "TUNE" (shape input) (at 0 60 0)
+  (hierarchical_label "NODE_B" (shape input) (at 50 220 0)
+    (fields_autoplaced)
+    (font (size 1.27 1.27) (thickness 0.254))
+  )
+  (hierarchical_label "V_tune" (shape input) (at 50 240 0)
     (fields_autoplaced)
     (font (size 1.27 1.27) (thickness 0.254))
   )
   ;; ──────────────────────────────────────────────
-  ;;  Hierarchical Labels — OUTPUT
+  ;;  Hierarchical Labels — GND
   ;; ──────────────────────────────────────────────
-  (hierarchical_label "LC_OUT" (shape output) (at 200 50 180)
+  (hierarchical_label "GND" (shape bidirectional) (at 300 50 90)
     (fields_autoplaced)
     (font (size 1.27 1.27) (thickness 0.254))
   )
   ;; ──────────────────────────────────────────────
-  ;;  Hierarchical Labels — POWER
+  ;;  GLOBAL POWER PORTS
   ;; ──────────────────────────────────────────────
-  (hierarchical_label "VDD" (shape bidirectional) (at 50 100 90)
+  (symbol (lib_name "power") (entry_id "GLOBAL_GND")
+    (in_bom yes) (on_board yes)
+    (property (name "Reference") (value "#PWR001"))
+    (property (name "Value")   (value "GND"))
+    (property (name "Footprint") (value ""))
+    (property (name "Datasheet") (value ""))
+    (property (name "ki_keywords") (value "global-power"))
+    (at 300 50 0)
+    (uuid "lc01g000-0001-4001-g001-000000000001")
+    (pin (at 0 0 0) (uuid "lc01g000-0001-4001-g001-0000000000p1"))
+;; ──────────────────────────────────────────────
+  ;;  COMPONENT: VARACTOR DIODE — D_var1 (BB833, SOT-23)
+  ;; ──────────────────────────────────────────────
+  (symbol (lib_id "Device:D") (at 200 200 0) (unit 1)
+    (in_bom yes) (on_board yes)
+    (property (name "Reference") (value "D1"))
+    (property (name "Value")   (value "BB833"))
+    (property (name "Footprint") (value "Package_TO_SOT_SMD:SOT-23"))
+    (property (name "Datasheet") (value "https://www.infineon.com/dgdl/bb833.pdf"))
+    (property (name "ki_description") (value "Varactor diode BB833 SOT-23 tuning element"))
+    (uuid "lc01d001-0001-4001-d001-000000000001")
+    (pin (at 0 0 0) (uuid "lc01d001-0001-4001-d001-00000000p1a"))
+    (pin (at 0 100 0) (uuid "lc01d001-0001-4001-d001-00000000p1k"))
+  )
+  ;; ──────────────────────────────────────────────
+  ;;  COMPONENT: VARACTOR DIODE — D_var2 (BB833, SOT-23)
+  ;; ──────────────────────────────────────────────
+  (symbol (lib_id "Device:D") (at 200 250 0) (unit 1)
+    (in_bom yes) (on_board yes)
+    (property (name "Reference") (value "D2"))
+    (property (name "Value")   (value "BB833"))
+    (property (name "Footprint") (value "Package_TO_SOT_SMD:SOT-23"))
+    (property (name "Datasheet") (value "https://www.infineon.com/dgdl/bb833.pdf"))
+    (property (name "ki_description") (value "Varactor diode BB833 SOT-23 tuning element"))
+    (uuid "lc01d002-0002-4002-d002-000000000002")
+    (pin (at 0 0 0) (uuid "lc01d002-0002-4002-d002-00000000p2a"))
+    (pin (at 0 100 0) (uuid "lc01d002-0002-4002-d002-00000000p2k"))
+  )
+  ;; ──────────────────────────────────────────────
+  ;;  COMPONENT: HIGH-Q SMD INDUCTOR — L1 (100uH, 1008/0805 shielded)
+  ;; ──────────────────────────────────────────────
+  (symbol (lib_id "Device:L") (at 300 200 0) (unit 1)
+    (in_bom yes) (on_board yes)
+    (property (name "Reference") (value "L1"))
+    (property (name "Value")   (value "100uH"))
+    (property (name "Footprint") (value "Inductor_SMD:L_1008_2520Metric"))
+    (property (name "Datasheet") (value ""))
+    (property (name "ki_description") (value "High-Q shielded inductor 100 uH resonance tank"))
+    (uuid "lc01l001-0001-4001-l001-000000000001")
+    (pin (at 0 0 0) (uuid "lc01l001-0001-4001-l001-00000000p1a"))
+    (pin (at 0 100 0) (uuid "lc01l001-0001-4001-l001-00000000p1b"))
+  )
+  ;; ──────────────────────────────────────────────
+  ;;  NET LABELS
+  ;; ──────────────────────────────────────────────
+  (label "LC_MID" (at 250 225 0)
     (fields_autoplaced)
-    (font (size 1.27 1.27) (thickness 0.254))
-  )
-  (hierarchical_label "VSS" (shape bidirectional) (at 70 100 90)
-    (fields_autoplaced)
-    (font (size 1.27 1.27) (thickness 0.254))
-  )
-  (hierarchical_label "GND" (shape bidirectional) (at 90 100 90)
-    (fields_autoplaced)
+    (uuid "lc01n001-0001-4001-n001-000000000001")
     (font (size 1.27 1.27) (thickness 0.254))
   )
   ;; ──────────────────────────────────────────────
-  ;;  Symbol & Schematic Body Placeholder
+  ;;  WIRES
   ;; ──────────────────────────────────────────────
-  ;; (Tunable inductor / capacitor network symbols
-  ;;  will be placed in the detailed design phase.)
+  ;; NODE_A -> D1 anode
+  (wire (pts (100 200) (200 200))
+    (stroke (width 0.1524) (type default) (color 0 0 0 0))
+    (uuid "lc01w001-0001-4001-w001-000000000001")
+  )
+  ;; NODE_B -> D2 anode
+  (wire (pts (100 220) (200 250))
+    (stroke (width 0.1524) (type default) (color 0 0 0 0))
+    (uuid "lc01w002-0002-4002-w002-000000000002")
+  )
+  ;; D1 cathode + D2 cathode -> LC_MID node
+  (wire (pts (200 300) (200 350))
+    (stroke (width 0.1524) (type default) (color 0 0 0 0))
+    (uuid "lc01w003-0003-4003-w003-000000000003")
+  )
+  (wire (pts (200 300) (250 300))
+    (stroke (width 0.1524) (type default) (color 0 0 0 0))
+    (uuid "lc01w004-0004-4004-w004-000000000004")
+  )
+  (wire (pts (250 300) (250 200))
+    (stroke (width 0.1524) (type default) (color 0 0 0 0))
+    (uuid "lc01w005-0005-4005-w005-000000000005")
+  )
+  ;; LC_MID -> L1
+  (wire (pts (250 225) (300 200))
+    (stroke (width 0.1524) (type default) (color 0 0 0 0))
+    (uuid "lc01w006-0006-4006-w006-000000000006")
+  )
+  ;; V_tune -> LC_MID (bias voltage for varactors)
+  (wire (pts (100 240) (250 240))
+    (stroke (width 0.1524) (type default) (color 0 0 0 0))
+    (uuid "lc01w007-0007-4007-w007-000000000007")
+  )
+  ;; L1 bottom -> GND
+  (wire (pts (300 300) (300 350))
+    (stroke (width 0.1524) (type default) (color 0 0 0 0))
+    (uuid "lc01w008-0008-4008-w008-000000000008")
+  )
+  (wire (pts (300 350) (300 100))
+    (stroke (width 0.1524) (type default) (color 0 0 0 0))
+    (uuid "lc01w009-0009-4009-w009-000000000009")
+  )
 )
+  )

Commit message: test(hardware): automate KiCad 10 schematic ERC validation and resolve power flag issues
Parts:
- added ? (x2): (no value), symbol Device:D
- added ?: (no value), symbol Device:L
- ?: symbol (none) -> power:GND
Changed lines of the file:
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@@
   ;;  GLOBAL POWER PORTS
   ;; ──────────────────────────────────────────────
-  (symbol (lib_name "power") (entry_id "GLOBAL_GND")
+  (symbol (lib_id "power:GND") (unit 1)
     (in_bom yes) (on_board yes)
     (property (name "Reference") (value "#PWR001"))
@@
     (uuid "lc01g000-0001-4001-g001-000000000001")
     (pin (at 0 0 0) (uuid "lc01g000-0001-4001-g001-0000000000p1"))
-;; ──────────────────────────────────────────────
+  )
+  ;; ──────────────────────────────────────────────
   ;;  COMPONENT: VARACTOR DIODE — D_var1 (BB833, SOT-23)
   ;; ──────────────────────────────────────────────
@@
   )
 )
-  )

Commit message: fix(hardware): fully migrate schematics to native KiCad 10 syntax and pass ERC
Parts:
- removed ? (x2): (no value), symbol Device:D
- removed ?: (no value), symbol power:GND
- removed ?: (no value), symbol Device:L
- added D2: BB833, Package_TO_SOT_SMD:SOT-23, symbol Device:D
- added L1: 100uH, Inductor_SMD:L_1008_2520Metric, symbol Device:L
Other:
- company: AdEx Resonant Brain Project -> Test
- title: LC Bridge Cell — Tunable Resonance Coupling -> Full Test3
Changed lines of the file:
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@@
-(kicad_sch (version 20240116) (generator "adex-resonant-brain")
+(kicad_sch (version 20240116) (generator "test")
   (paper "A4")
-  (title_block
-    (title "LC Bridge Cell — Tunable Resonance Coupling")
-    (date "2026-09-06")
-    (rev "1.0")
-    (company "AdEx Resonant Brain Project")
+  (title_block (title "Full Test3") (date "2026-09-06") (rev "1.0") (company "Test"))
+  (symbol
+    (lib_id "power:GND")
+    (at 50 50 0)
+    (unit 1)
+    (exclude_from_sim no)
+    (in_bom yes)
+    (on_board yes)
+    (dnp no)
+    (property "Reference" "#PWR001"
+      (at 50 50 0)
+      (effects (font (size 1.27 1.27)))
+    )
+    (property "Value" "GND"
+      (at 50 50 0)
+      (effects (font (size 1.27 1.27)))
+    )
+    (property "Footprint" ""
+      (at 50 50 0)
+      (effects (font (size 1.27 1.27)) (hide yes))
+    )
+    (property "Datasheet" ""
+      (at 50 50 0)
+      (effects (font (size 1.27 1.27)) (hide yes))
+    )
+    (property "ki_keywords" "global-power"
+      (at 50 50 0)
+      (effects (font (size 1.27 1.27)) (hide yes))
+    )
   )
-  ;; ──────────────────────────────────────────────
-  ;;  Hierarchical Labels — INPUT
-  ;; ──────────────────────────────────────────────
-  (hierarchical_label "NODE_A" (shape input) (at 50 200 0)
-    (fields_autoplaced)
-    (font (size 1.27 1.27) (thickness 0.254))
+  (symbol
+    (lib_id "Device:L")
+    (at 300 200 0)
+    (unit 1)
+    (exclude_from_sim no)
+    (in_bom yes)
+    (on_board yes)
+    (dnp no)
+    (property "Reference" "L1"
+      (at 300 200 0)
+      (effects (font (size 1.27 1.27)))
+    )
+    (property "Value" "100uH"
+      (at 300 200 0)
+      (effects (font (size 1.27 1.27)))
+    )
+    (property "Footprint" "Inductor_SMD:L_1008_2520Metric"
+      (at 300 200 0)
+      (effects (font (size 1.27 1.27)) (hide yes))
+    )
+    (property "Datasheet" ""
+      (at 300 200 0)
+      (effects (font (size 1.27 1.27)) (hide yes))
+    )
+    (property "ki_description" "High-Q inductor 100 uH"
+      (at 300 200 0)
+      (effects (font (size 1.27 1.27)))
+    )
   )
-  (hierarchical_label "NODE_B" (shape input) (at 50 220 0)
-    (fields_autoplaced)
-    (font (size 1.27 1.27) (thickness 0.254))
-  )
-  (hierarchical_label "V_tune" (shape input) (at 50 240 0)
-    (fields_autoplaced)
-    (font (size 1.27 1.27) (thickness 0.254))
-  )
-  ;; ──────────────────────────────────────────────
-  ;;  Hierarchical Labels — GND
-  ;; ──────────────────────────────────────────────
-  (hierarchical_label "GND" (shape bidirectional) (at 300 50 90)
-    (fields_autoplaced)
-    (font (size 1.27 1.27) (thickness 0.254))
-  )
-  ;; ──────────────────────────────────────────────
-  ;;  GLOBAL POWER PORTS
-  ;; ──────────────────────────────────────────────
-  (symbol (lib_id "power:GND") (unit 1)
-    (in_bom yes) (on_board yes)
-    (property (name "Reference") (value "#PWR001"))
-    (property (name "Value")   (value "GND"))
-    (property (name "Footprint") (value ""))
-    (property (name "Datasheet") (value ""))
-    (property (name "ki_keywords") (value "global-power"))
-    (at 300 50 0)
-    (uuid "lc01g000-0001-4001-g001-000000000001")
-    (pin (at 0 0 0) (uuid "lc01g000-0001-4001-g001-0000000000p1"))
-  )
-  ;; ──────────────────────────────────────────────
-  ;;  COMPONENT: VARACTOR DIODE — D_var1 (BB833, SOT-23)
-  ;; ──────────────────────────────────────────────
-  (symbol (lib_id "Device:D") (at 200 200 0) (unit 1)
-    (in_bom yes) (on_board yes)
-    (property (name "Reference") (value "D1"))
-    (property (name "Value")   (value "BB833"))
-    (property (name "Footprint") (value "Package_TO_SOT_SMD:SOT-23"))
-    (property (name "Datasheet") (value "https://www.infineon.com/dgdl/bb833.pdf"))
-    (property (name "ki_description") (value "Varactor diode BB833 SOT-23 tuning element"))
-    (uuid "lc01d001-0001-4001-d001-000000000001")
-    (pin (at 0 0 0) (uuid "lc01d001-0001-4001-d001-00000000p1a"))
-    (pin (at 0 100 0) (uuid "lc01d001-0001-4001-d001-00000000p1k"))
-  )
-  ;; ──────────────────────────────────────────────
-  ;;  COMPONENT: VARACTOR DIODE — D_var2 (BB833, SOT-23)
-  ;; ──────────────────────────────────────────────
-  (symbol (lib_id "Device:D") (at 200 250 0) (unit 1)
-    (in_bom yes) (on_board yes)
-    (property (name "Reference") (value "D2"))
-    (property (name "Value")   (value "BB833"))
-    (property (name "Footprint") (value "Package_TO_SOT_SMD:SOT-23"))
-    (property (name "Datasheet") (value "https://www.infineon.com/dgdl/bb833.pdf"))
-    (property (name "ki_description") (value "Varactor diode BB833 SOT-23 tuning element"))
-    (uuid "lc01d002-0002-4002-d002-000000000002")
-    (pin (at 0 0 0) (uuid "lc01d002-0002-4002-d002-00000000p2a"))
-    (pin (at 0 100 0) (uuid "lc01d002-0002-4002-d002-00000000p2k"))
-  )
-  ;; ──────────────────────────────────────────────
-  ;;  COMPONENT: HIGH-Q SMD INDUCTOR — L1 (100uH, 1008/0805 shielded)
-  ;; ──────────────────────────────────────────────
-  (symbol (lib_id "Device:L") (at 300 200 0) (unit 1)
-    (in_bom yes) (on_board yes)
-    (property (name "Reference") (value "L1"))
-    (property (name "Value")   (value "100uH"))
-    (property (name "Footprint") (value "Inductor_SMD:L_1008_2520Metric"))
-    (property (name "Datasheet") (value ""))
-    (property (name "ki_description") (value "High-Q shielded inductor 100 uH resonance tank"))
-    (uuid "lc01l001-0001-4001-l001-000000000001")
-    (pin (at 0 0 0) (uuid "lc01l001-0001-4001-l001-00000000p1a"))
-    (pin (at 0 100 0) (uuid "lc01l001-0001-4001-l001-00000000p1b"))
-  )
-  ;; ──────────────────────────────────────────────
-  ;;  NET LABELS
-  ;; ──────────────────────────────────────────────
-  (label "LC_MID" (at 250 225 0)
-    (fields_autoplaced)
-    (uuid "lc01n001-0001-4001-n001-000000000001")
-    (font (size 1.27 1.27) (thickness 0.254))
-  )
-  ;; ──────────────────────────────────────────────
-  ;;  WIRES
-  ;; ──────────────────────────────────────────────
-  ;; NODE_A -> D1 anode
-  (wire (pts (100 200) (200 200))
-    (stroke (width 0.1524) (type default) (color 0 0 0 0))
-    (uuid "lc01w001-0001-4001-w001-000000000001")
-  )
-  ;; NODE_B -> D2 anode
-  (wire (pts (100 220) (200 250))
-    (stroke (width 0.1524) (type default) (color 0 0 0 0))
-    (uuid "lc01w002-0002-4002-w002-000000000002")
-  )
-  ;; D1 cathode + D2 cathode -> LC_MID node
-  (wire (pts (200 300) (200 350))
-    (stroke (width 0.1524) (type default) (color 0 0 0 0))
-    (uuid "lc01w003-0003-4003-w003-000000000003")
-  )
-  (wire (pts (200 300) (250 300))
-    (stroke (width 0.1524) (type default) (color 0 0 0 0))
-    (uuid "lc01w004-0004-4004-w004-000000000004")
-  )
-  (wire (pts (250 300) (250 200))
-    (stroke (width 0.1524) (type default) (color 0 0 0 0))
-    (uuid "lc01w005-0005-4005-w005-000000000005")
-  )
-  ;; LC_MID -> L1
-  (wire (pts (250 225) (300 200))
-    (stroke (width 0.1524) (type default) (color 0 0 0 0))
-    (uuid "lc01w006-0006-4006-w006-000000000006")
-  )
-  ;; V_tune -> LC_MID (bias voltage for varactors)
-  (wire (pts (100 240) (250 240))
-    (stroke (width 0.1524) (type default) (color 0 0 0 0))
-    (uuid "lc01w007-0007-4007-w007-000000000007")
-  )
-  ;; L1 bottom -> GND
-  (wire (pts (300 300) (300 350))
-    (stroke (width 0.1524) (type default) (color 0 0 0 0))
-    (uuid "lc01w008-0008-4008-w008-000000000008")
-  )
-  (wire (pts (300 350) (300 100))
-    (stroke (width 0.1524) (type default) (color 0 0 0 0))
-    (uuid "lc01w009-0009-4009-w009-000000000009")
+  (hierarchical_label "NODE_A" (shape input) (at 50 200 0) (effects (font (size 1.27 1.27))))
+  (hierarchical_label "NODE_B" (shape input) (at 50 220 0) (effects (font (size 1.27 1.27))))
+  (hierarchical_label "V_tune" (shape input) (at 50 240 0) (effects (font (size 1.27 1.27))))
+  (hierarchical_label "GND" (shape bidirectional) (at 300 50 90) (effects (font (size 1.27 1.27))))
+  (label "LC_MID" (at 250 225 0) (effects (font (size 1.27 1.27))))
+  (symbol
+    (lib_id "Device:D")
+    (at 200 250 0)
+    (unit 1)
+    (exclude_from_sim no)
+    (in_bom yes)
+    (on_board yes)
+    (dnp no)
+    (property "Reference" "D2"
+      (at 200 250 0)
+      (effects (font (size 1.27 1.27)))
+    )
+    (property "Value" "BB833"
+      (at 200 250 0)
+      (effects (font (size 1.27 1.27)))
+    )
+    (property "Footprint" "Package_TO_SOT_SMD:SOT-23"
+      (at 200 250 0)
+      (effects (font (size 1.27 1.27)) (hide yes))
+    )
+    (property "Datasheet" "https://www.infineon.com/dgdl/bb833.pdf"
+      (at 200 250 0)
+      (effects (font (size 1.27 1.27)) (hide yes))
+    )
+    (property "ki_description" "Varactor diode BB833 SOT-23 tuning element"
+      (at 200 250 0)
+      (effects (font (size 1.27 1.27)))
+    )
   )
 )

Commit message: feat(hardware): assign SMD footprints and generate 4-layer KiCad 10 PCB layout
Other:
- company: Test -> AdEx Resonant Brain Project
- title: Full Test3 -> LC Bridge Cell — Resonant LC Tank with Varactor Tuning
Changed lines of the file:
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@@
-(kicad_sch (version 20240116) (generator "test")
+(kicad_sch (version 20240116) (generator "adex-resonant-brain")
   (paper "A4")
-  (title_block (title "Full Test3") (date "2026-09-06") (rev "1.0") (company "Test"))
+  (title_block
+    (title "LC Bridge Cell — Resonant LC Tank with Varactor Tuning")
+    (date "2026-09-06")
+    (rev "1.0")
+    (company "AdEx Resonant Brain Project")
+  )
   (symbol
-    (lib_id "power:GND")
+    (lib_id "custom_power:GND")
     (at 50 50 0)
     (unit 1)
